File: Catwan_sensorwater/Catwan_sensorwater.sch (KiCad schematic (older format))
At the start: 7 parts, among them U1 AP2127N-1.0

Commit message: Agregue ATSAMD Y LORA
Parts:
- removed C1, C3: 10uf, Capacitor_SMD:C_0805_2012Metric_Pad1.15x1.40mm_HandSolder, symbol Device:C
- removed R?: R, symbol Device:R
- added AE?: Antenna_Shield, symbol Device:Antenna_Shield
- added C? (x2): 10uf, Capacitor_SMD:C_0805_2012Metric_Pad1.15x1.40mm_HandSolder, symbol Device:C
- added C?: 0.1uf, Capacitor_SMD:C_0805_2012Metric_Pad1.15x1.40mm_HandSolder, symbol Device:C
- added J?: Conn_01x04_Female, symbol Connector:Conn_01x04_Female
- added J?: Conn_01x03_Female, symbol Connector:Conn_01x03_Female
- added J?: USB_B, symbol Connector:USB_B
- added SW?: SW_DPST_x2, symbol Switch:SW_DPST_x2
- added U?: ATSAMD21E18A-MU, QFN50P500X500X100-33N, symbol electroniccats:ATSAMD21E18A-MU
- added U?: RFM95W-868S2, symbol RF_AM_FM:RFM95W-868S2
- C?: value C -> 1uf
Connections:
- net labels added: D+, D-, DIO1, DIO2, DIO5, MIS0, MOSI, RFM_RST, SCK, SS, SWCLK, SWDIO, X
- wire segments 15 -> 45

Commit message: SENSORES, MULTIPLEXOR
Parts:
- removed C?: C, symbol Device:C
- added D? (x4): D_Zener, symbol Device:D_Zener
Connections:
- net labels added: DI2, DI3, DIO0, DO1, DO2, DO3, RST, Rx, Rx_LED, Tx, VBUS, x
- wire segments 45 -> 63
Other:
- note added: "MICROCONTROLLER"
- note added: "MODULATION LORA\n"
- note added: "POWER SUPPLY"
- note added: "SENSORES\n"

Commit message: Multiplexor casi listo.
Parts:
- added J? (x2): Conn_01x02, symbol Connector_Generic:Conn_01x02
- added R? (x2): R, symbol Device:R
- added U?: 74HC4052, symbol electroniccats:74HC4052
Connections:
- wire segments 63 -> 94
Changed lines of the file:
@@
 L Device:D_Zener D?
 U 1 1 5BB6CA62
-P 6468 5112
-F 0 "D?" H 6468 5328 50  0000 C CNN
-F 1 "D_Zener" H 6468 5237 50  0000 C CNN
-F 2 "" H 6468 5112 50  0001 C CNN
-F 3 "~" H 6468 5112 50  0001 C CNN
-	1    6468 5112
+P 6268 4956
+F 0 "D?" H 6268 5172 50  0000 C CNN
+F 1 "D_Zener" H 6268 5081 50  0000 C CNN
+F 2 "" H 6268 4956 50  0001 C CNN
+F 3 "~" H 6268 4956 50  0001 C CNN
+	1    6268 4956
 	1    0    0    -1
 $EndComp
@@
 L Device:D_Zener D?
 U 1 1 5BB6CB06
-P 6444 5502
-F 0 "D?" H 6444 5718 50  0000 C CNN
-F 1 "D_Zener" H 6444 5627 50  0000 C CNN
-F 2 "" H 6444 5502 50  0001 C CNN
-F 3 "~" H 6444 5502 50  0001 C CNN
-	1    6444 5502
+P 6264 5080
+F 0 "D?" H 6370 5154 50  0000 C CNN
+F 1 "D_Zener" H 6472 5026 50  0000 C CNN
+F 2 "" H 6264 5080 50  0001 C CNN
+F 3 "~" H 6264 5080 50  0001 C CNN
+	1    6264 5080
 	1    0    0    -1
 $EndComp
@@
 L Device:D_Zener D?
 U 1 1 5BB6CB9A
-P 6438 5958
-F 0 "D?" H 6438 6174 50  0000 C CNN
-F 1 "D_Zener" H 6438 6083 50  0000 C CNN
-F 2 "" H 6438 5958 50  0001 C CNN
-F 3 "~" H 6438 5958 50  0001 C CNN
-	1    6438 5958
+P 6260 5258
+F 0 "D?" H 6364 5310 50  0000 C CNN
+F 1 "D_Zener" H 6472 5196 50  0000 C CNN
+F 2 "" H 6260 5258 50  0001 C CNN
+F 3 "~" H 6260 5258 50  0001 C CNN
+	1    6260 5258
 	1    0    0    -1
 $EndComp
@@
 L Device:D_Zener D?
 U 1 1 5BB6CC0E
-P 6408 6366
-F 0 "D?" H 6408 6582 50  0000 C CNN
-F 1 "D_Zener" H 6408 6491 50  0000 C CNN
-F 2 "" H 6408 6366 50  0001 C CNN
-F 3 "~" H 6408 6366 50  0001 C CNN
-	1    6408 6366
+P 6258 5454
+F 0 "D?" H 6364 5500 50  0000 C CNN
+F 1 "D_Zener" H 6460 5384 50  0000 C CNN
+F 2 "" H 6258 5454 50  0001 C CNN
+F 3 "~" H 6258 5454 50  0001 C CNN
+	1    6258 5454
 	1    0    0    -1
 $EndComp
@@
 L power:GND #PWR?
 U 1 1 5BB6D389
-P 4944 6438
-F 0 "#PWR?" H 4944 6188 50  0001 C CNN
-F 1 "GND" V 4949 6310 50  0000 R CNN
-F 2 "" H 4944 6438 50  0001 C CNN
-F 3 "" H 4944 6438 50  0001 C CNN
-	1    4944 6438
+P 4822 5558
+F 0 "#PWR?" H 4822 5308 50  0001 C CNN
+F 1 "GND" V 4827 5430 50  0000 R CNN
+F 2 "" H 4822 5558 50  0001 C CNN
+F 3 "" H 4822 5558 50  0001 C CNN
+	1    4822 5558
 	1    0    0    -1
 $EndComp
+$Comp
+L electroniccats:74HC4052 U?
+U 1 1 5BB40CAB
+P 5404 5256
+F 0 "U?" H 5404 5826 50  0000 C CNN
+F 1 "74HC4052" H 5404 5735 50  0000 C CNN
+F 2 "" H 5404 5256 50  0001 C CNN
+F 3 "Sig/Phil 74hc4052d Smd 50/Tube" H 5404 5256 50  0001 L BNN
+F 4 "NXP Semiconductors" H 5404 5256 50  0001 L BNN "Campo4"
+F 5 "DIP-16 NXP Semiconductors" H 5404 5256 50  0001 L BNN "Campo5"
+F 6 "Unavailable" H 5404 5256 50  0001 L BNN "Campo6"
+F 7 "74HC4052" H 5404 5256 50  0001 L BNN "Campo7"
+F 8 "None" H 5404 5256 50  0001 L BNN "Campo8"
+	1    5404 5256
+	1    0    0    -1
+$EndComp
+Wire Wire Line
+	6118 4956 5804 4956
+Wire Wire Line
+	5804 5056 6094 5056
+Wire Wire Line
+	6094 5056 6094 5080
+Wire Wire Line
+	6094 5080 6114 5080
+Wire Wire Line
+	5804 5156 6068 5156
+Wire Wire Line
+	6068 5156 6068 5258
+Wire Wire Line
+	6068 5258 6110 5258
+Wire Wire Line
+	5804 5256 6026 5256
+Wire Wire Line
+	6026 5256 6026 5454
+Wire Wire Line
+	6026 5454 6108 5454
+$Comp
+L Connector_Generic:Conn_01x02 J?
+U 1 1 5BB53012
+P 6902 4952
+F 0 "J?" H 6982 4944 50  0000 L CNN
+F 1 "Conn_01x02" H 6982 4853 50  0000 L CNN
+F 2 "" H 6902 4952 50  0001 C CNN
+F 3 "~" H 6902 4952 50  0001 C CNN
+	1    6902 4952
+	1    0    0    -1
+$EndComp
+Wire Wire Line
+	6418 4956 6682 4956
+Wire Wire Line
+	6682 4956 6682 4952
+Wire Wire Line
+	6682 4952 6702 4952
+Wire Wire Line
+	6414 5080 6682 5080
+Wire Wire Line
+	6682 5080 6682 5052
+Wire Wire Line
+	6682 5052 6702 5052
+$Comp
+L Connector_Generic:Conn_01x02 J?
+U 1 1 5BB578EE
+P 6912 5262
+F 0 "J?" H 6992 5254 50  0000 L CNN
+F 1 "Conn_01x02" H 6992 5163 50  0000 L CNN
+F 2 "" H 6912 5262 50  0001 C CNN
+F 3 "~" H 6912 5262 50  0001 C CNN
+	1    6912 5262
+	1    0    0    -1
+$EndComp
+Wire Wire Line
+	6410 5258 6692 5258
+Wire Wire Line
+	6692 5258 6692 5262
+Wire Wire Line
+	6692 5262 6712 5262
+Wire Wire Line
+	6408 5454 6670 5454
+Wire Wire Line
+	6670 5454 6670 5362
+Wire Wire Line
+	6670 5362 6712 5362
+$Comp
+L power:+3.3V #PWR?
+U 1 1 5BB5F6BD
+P 4816 4956
+F 0 "#PWR?" H 4816 4806 50  0001 C CNN
+F 1 "+3.3V" H 4831 5129 50  0000 C CNN
+F 2 "" H 4816 4956 50  0001 C CNN
+F 3 "" H 4816 4956 50  0001 C CNN
+	1    4816 4956
+	0    -1   -1   0
+$EndComp
+Wire Wire Line
+	4816 4956 5004 4956
+Wire Wire Line
+	4822 5558 4822 5556
+Wire Wire Line
+	4822 5556 5004 5556
+$Comp
+L Device:R R?
+U 1 1 5BB67877
+P 6124 5710
+F 0 "R?" H 6194 5756 50  0000 L CNN
+F 1 "R" H 6194 5665 50  0000 L CNN
+F 2 "" V 6054 5710 50  0001 C CNN
+F 3 "~" H 6124 5710 50  0001 C CNN
+	1    6124 5710
+	1    0    0    -1
+$EndComp
+$Comp
+L Device:R R?
+U 1 1 5BB6791D
+P 6028 5712
+F 0 "R?" H 5886 5784 50  0000 L CNN
+F 1 "R" H 5926 5658 50  0000 L CNN
+F 2 "" V 5958 5712 50  0001 C CNN
+F 3 "~" H 6028 5712 50  0001 C CNN
+	1    6028 5712
+	1    0    0    -1
+$EndComp
+Wire Wire Line
+	5804 5356 6000 5356
+Wire Wire Line
+	6000 5356 6000 5530
+Wire Wire Line
+	6000 5530 6028 5530
+Wire Wire Line
+	6124 5530 6124 5560
+Wire Wire Line
+	6028 5562 6028 5530
+Connection ~ 6028 5530
+Wire Wire Line
+	6028 5530 6124 5530
 $EndSCHEMATC

Commit message: asignación huellas
Parts:
- removed R? (x2): R, symbol Device:R
- added D1, D2: D_Zener, symbol Device:D_Zener
- added J4: Conn_01x02, symbol Connector_Generic:Conn_01x02
- added R1, R2: R, Resistor_SMD:R_0805_2012Metric_Pad1.15x1.40mm_HandSolder, symbol Device:R
- C3: renamed from C?; footprint (none) -> Capacitor_SMD:C_0805_2012Metric_Pad1.15x1.40mm_HandSolder
- SW1: renamed from SW?; footprint (none) -> Button_Switch_SMD:SW_SPST_B3U-1000P
- gave numbers to parts that had none: 16
Connections:
- net labels added: Y
- wire segments 94 -> 113

Commit message: batería agregada.
Parts:
- added C6: 10uf, Capacitor_SMD:C_0805_2012Metric_Pad1.15x1.40mm_HandSolder, symbol Device:C
- added D10, D7: LED, symbol Device:LED
- added D8, D9: D_Zener, symbol Device:D_Zener
- added J7: BATT, symbol Connector_Generic:Conn_01x02
- added R3, R4: 10K, symbol Device:R
- added R5, R6: 1K, symbol Device:R
- added U5: MCP73831-4-OT, Package_TO_SOT_SMD:SOT-23-5, symbol Battery_Management:MCP73831-4-OT
Connections:
- net labels added: BAT
- wire segments 113 -> 143
Other:
- note added: "Charger"

Commit message: huellas
Cambios
Parts:
- J1, J2, J4, J5, J6: footprint (none) -> TerminalBlock_Phoenix:TerminalBlock_Phoenix_PT-1,5-2-3.5-H_1x02_P3.50mm_Horizontal
- R3, R4, R5, R6: footprint (none) -> Resistor_SMD:R_0815_2038Metric_Pad1.53x4.00mm_HandSolder
Other:
- moved on the sheet: U5

Commit message: add s0 s1 ans enable in multiplexer
Parts:
- J4: value Conn_01x02 -> SENSOR 3
- J5: value Conn_01x02 -> SENSOR 1
- J6: value Conn_01x02 -> SENSOR 2
- R1, R2: value R -> 4K7
Connections:
- net labels added: EN, S0, S1
- wire segments 143 -> 129
- no-connect marks 0 -> 2

Commit message: Edit ATSAMD separate pin 10 and 28 an no connected
Parts:
- J1: value Conn_01x04_Female -> SWD
- J2: value Conn_01x03_Female -> Serial
- SW1: value SW_DPST_x2 -> RST
Connections:
- net labels removed: RST
- wire segments 129 -> 132
- no-connect marks 2 -> 4
