File: Catwan_sensorwater/_autosave-Catwan_sensorwater.kicad_pcb (KiCad board)
At the start: 2 copper layers, 64 x 45 mm, 41 parts, among them J1 SENSOR 1, J10 VSP, J2 SENSOR 2, J3 SENSOR 3, J4 BATT, J5 USB_B, J6 Conn_01x04, J7 Conn_01x03, J8 Conn_01x03_Female, J9 SENSOR 4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

Commit message: clear schematic
Parts:
- removed D8, D9: D_Zener, Diode_SMD:D_SOD-123
- added D1: D_Schottky, Diode_SMD:D_0805_2012Metric_Pad1.15x1.40mm_HandSolder, B.Cu at (148.5, 92.0)
- moved J4 10.3 mm to (152.2, 85.0)
- moved J10 8.24 mm to (162.3, 84.8)
- moved C9 0.95 mm to (154.2, 99.2)
- moved C10 0.88 mm to (154.0, 96.3)
- moved U4 0.43 mm to (154.5, 92.8), turned to 180 degrees
Connections:
- AE1 pad 4: GND -> (no net)
- AE1 pad 5: GND -> (no net)
- AE1 pad E: GND -> (no net)
- C4 pad 1: +3V3 -> Net-(C4-Pad1)
- J10 pad 2: VCC -> /Vsp
- U1 pad 3: +3V3 -> VCC
