File: Hardware/Catwan_Farmer.sch (KiCad schematic (older format))
At the start: 47 parts, among them J1 SENSOR 1, J10 VSP, J2 SENSOR 2, J3 SENSOR 3, J4 BATT, J5 USB_B, J6 Conn_01x04, J7 DHT22, J9 SENSOR 4, Q1 BSS214NW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

Commit message: Value Mosfet
Parts:
- Q1, Q2, Q3, Q4: value BSS214NW -> 2N7002
- U2: symbol Catwan_Farmer-rescue:ATSAMD21E18A-MU-electroniccats-Catwan_sensorwater-rescue-Catwan_sensorwater-rescue-Catwan_sensorwater-rescue-Catwan_sensorwater-rescue-Catwan_sensorwater-rescue -> Catwan_Farmer-rescue:ATSAMD21E18A-MU-electroniccats-Catwan_sensorwater-rescue-Catwan_sensorwater-rescue-Catwan_sensorwater-rescue-Catwan_sensorwater-rescue-Catwan_sensorwater-rescue-Catwan_Farmer-rescue
Changed lines of the file:
@@
 $EndComp
 $Comp
-L Catwan_Farmer-rescue:ATSAMD21E18A-MU-electroniccats-Catwan_sensorwater-rescue-Catwan_sensorwater-rescue-Catwan_sensorwater-rescue-Catwan_sensorwater-rescue-Catwan_sensorwater-rescue U2
+L Catwan_Farmer-rescue:ATSAMD21E18A-MU-electroniccats-Catwan_sensorwater-rescue-Catwan_sensorwater-rescue-Catwan_sensorwater-rescue-Catwan_sensorwater-rescue-Catwan_sensorwater-rescue-Catwan_Farmer-rescue U2
 U 1 1 5BAD6569
 P 2500 2160
@@
 P 8905 6046
 F 0 "Q1" H 9062 6158 50  0000 L CNN
-F 1 "BSS214NW" H 8544 5805 50  0000 L CNN
+F 1 "2N7002" H 8544 5805 50  0000 L CNN
 F 2 "Package_TO_SOT_SMD:SOT-23" H 9105 5971 50  0001 L CIN
 F 3 "https://www.infineon.com/dgdl/Infineon-BSS214NW-DS-v02_02-en.pdf?fileId=db3a30431b3e89eb011b695aebc01bde" H 8905 6046 50  0001 L CNN
@@
 P 9450 6038
 F 0 "Q2" H 9606 6146 50  0000 L CNN
-F 1 "BSS214NW" H 9110 5809 50  0000 L CNN
+F 1 "2N7002" H 9110 5809 50  0000 L CNN
 F 2 "Package_TO_SOT_SMD:SOT-23" H 9650 5963 50  0001 L CIN
 F 3 "https://www.infineon.com/dgdl/Infineon-BSS214NW-DS-v02_02-en.pdf?fileId=db3a30431b3e89eb011b695aebc01bde" H 9450 6038 50  0001 L CNN
@@
 P 9974 6048
 F 0 "Q3" H 10121 6166 50  0000 L CNN
-F 1 "BSS214NW" H 9634 5819 50  0000 L CNN
+F 1 "2N7002" H 9634 5819 50  0000 L CNN
 F 2 "Package_TO_SOT_SMD:SOT-23" H 10174 5973 50  0001 L CIN
 F 3 "https://www.infineon.com/dgdl/Infineon-BSS214NW-DS-v02_02-en.pdf?fileId=db3a30431b3e89eb011b695aebc01bde" H 9974 6048 50  0001 L CNN
@@
 P 10460 6049
 F 0 "Q4" H 10642 6173 50  0000 L CNN
-F 1 "BSS214NW" H 10120 5820 50  0000 L CNN
+F 1 "2N7002" H 10120 5820 50  0000 L CNN
 F 2 "Package_TO_SOT_SMD:SOT-23" H 10660 5974 50  0001 L CIN
 F 3 "https://www.infineon.com/dgdl/Infineon-BSS214NW-DS-v02_02-en.pdf?fileId=db3a30431b3e89eb011b695aebc01bde" H 10460 6049 50  0001 L CNN

Commit message: add LED and sens voltage
Parts:
- U2: symbol Catwan_Farmer-rescue:ATSAMD21E18A-MU-electroniccats-Catwan_sensorwater-rescue-Catwan_sensorwater-rescue-Catwan_sensorwater-rescue-Catwan_sensorwater-rescue-Catwan_sensorwater-rescue-Catwan_Farmer-rescue -> Catwan_Farmer-rescue:ATSAMD21E18A-MU-electroniccats-Catwan_sensorwater-rescue-Catwan_sensorwater-rescue-Catwan_sensorwater-rescue-Catwan_sensorwater-rescue-Catwan_sensorwater-rescue-Catwan_Farmer-rescue-Catwan_Farmer-rescue
- U5: symbol electroniccats:74HC4052 -> Catwan_Farmer-rescue:74HC4052-electroniccats
Connections:
- net labels added: LED, SEN_X, SEN_Y
- wire segments 180 -> 181
- no-connect marks 7 -> 4
Changed lines of the file:
@@
 EESchema Schematic File Version 4
 LIBS:Catwan_Farmer-cache
-EELAYER 26 0
+EELAYER 29 0
 EELAYER END
 $Descr A4 11693 8268
@@
 Text Label 3200 2260 0    50   ~ 0
 EN
-NoConn ~ 1800 2460
 Text Label 1800 1860 2    50   ~ 0
 SENS_X
@@
 	3279 3754 3279 3982
 $Comp
-L electroniccats:74HC4052 U5
+L Catwan_Farmer-rescue:74HC4052-electroniccats U5
 U 1 1 5C0415EA
 P 8414 5185
@@
 $EndComp
 $Comp
-L Catwan_Farmer-rescue:ATSAMD21E18A-MU-electroniccats-Catwan_sensorwater-rescue-Catwan_sensorwater-rescue-Catwan_sensorwater-rescue-Catwan_sensorwater-rescue-Catwan_sensorwater-rescue-Catwan_Farmer-rescue U2
+L Catwan_Farmer-rescue:ATSAMD21E18A-MU-electroniccats-Catwan_sensorwater-rescue-Catwan_sensorwater-rescue-Catwan_sensorwater-rescue-Catwan_sensorwater-rescue-Catwan_sensorwater-rescue-Catwan_Farmer-rescue-Catwan_Farmer-rescue U2
 U 1 1 5BAD6569
 P 2500 2160
@@
 Connection ~ 970  2020
 Wire Wire Line
-	770  2290 870  2290
-Wire Wire Line
 	970  2290 970  2270
-Wire Wire Line
-	870  2290 870  2360
-Connection ~ 870  2290
-Wire Wire Line
-	870  2290 970  2290
-$Comp
-L power:GND #PWR010
-U 1 1 5C7439DB
-P 870 2360
-F 0 "#PWR010" H 870 2110 50  0001 C CNN
-F 1 "GND" H 875 2187 50  0000 C CNN
-F 2 "" H 870 2360 50  0001 C CNN
-F 3 "" H 870 2360 50  0001 C CNN
-	1    870  2360
-	1    0    0    -1
-$EndComp
 Text Label 970  1840 0    50   ~ 0
 Y1
@@
 Wire Wire Line
 	1720 1460 1800 1460
-NoConn ~ 1800 2160
 NoConn ~ 1800 2260
-NoConn ~ 1800 2360
 Wire Wire Line
 	5020 7220 5020 7120
@@
 Wire Wire Line
 	9460 3620 9280 3620
+Wire Wire Line
+	770  2290 970  2290
+Wire Wire Line
+	1800 2460 1515 2460
+Wire Wire Line
+	1800 2360 1515 2360
+Wire Wire Line
+	1800 2160 1535 2160
+Text Label 1515 2460 0    50   ~ 0
+LED
+Text Label 1515 2360 0    50   ~ 0
+SEN_Y
+Text Label 1535 2160 0    50   ~ 0
+SEN_X
 $EndSCHEMATC

Commit message: change mosfet to zenner
Parts:
- removed Q1, Q2, Q3, Q4: 2N7002, Package_TO_SOT_SMD:SOT-23, symbol Transistor_FET:BSS214NW
- added D4, D5, D6, D8: AZ23C9V1, symbol Device:D_Zener_x2_ACom_KKA
- U3: symbol RF_AM_FM:RFM95W-868S2 -> Catwan_Farmer-rescue:RFM95W-868S2-RF_AM_FM
- U5: symbol Catwan_Farmer-rescue:74HC4052-electroniccats -> Catwan_Farmer-rescue:74HC4052-electroniccats-Catwan_Farmer-rescue
Connections:
- net GND: now also D4.3 (A), D5.3 (A), D6.3 (A), D8.3 (A)
- net at J1.1 (Pin_1), U5.12 (X0): now also D8.1 (K)
- net at J1.2 (Pin_2), U5.14 (X1): now also D8.2 (K)
- net at J2.1 (Pin_1), U5.15 (X2): now also D5.1 (K)
- net at J2.2 (Pin_2), U5.11 (X3): now also D5.2 (K)
- net at J9.1 (Pin_1), U5.2 (Y2): now also D4.1 (K)
- net at J9.2 (Pin_2), U5.4 (Y3): now also D4.2 (K)
- net at J3.1 (Pin_1), U5.1 (Y0): now also D6.1 (K)
- net at J3.2 (Pin_2), U5.5 (Y1): now also D6.2 (K)
Changed lines of the file:
@@
 Sheet 1 1
 Title "CatWAN"
-Date "2018-11-07"
-Rev "0.4"
+Date "2019-05-27"
+Rev "0.5"
 Comp "Electronic Cats"
 Comment1 "Montserrat Figueroa"
@@
 	2166 6480 2066 6480
 $Comp
-L RF_AM_FM:RFM95W-868S2 U3
+L Catwan_Farmer-rescue:RFM95W-868S2-RF_AM_FM U3
 U 1 1 5BAF85CF
 P 2066 5762
@@
 L power:GND #PWR0108
 U 1 1 5BE5CD63
-P 9005 6401
-F 0 "#PWR0108" H 9005 6151 50  0001 C CNN
-F 1 "GND" H 8877 6339 50  0000 C CNN
-F 2 "" H 9005 6401 50  0001 C CNN
-F 3 "" H 9005 6401 50  0001 C CNN
-	1    9005 6401
+P 9285 6405
+F 0 "#PWR0108" H 9285 6155 50  0001 C CNN
+F 1 "GND" H 9157 6343 50  0000 C CNN
+F 2 "" H 9285 6405 50  0001 C CNN
+F 3 "" H 9285 6405 50  0001 C CNN
+	1    9285 6405
 	1    0    0    -1
 $EndComp
@@
 L power:GND #PWR0109
 U 1 1 5BDCFBA0
-P 9550 6393
-F 0 "#PWR0109" H 9550 6143 50  0001 C CNN
-F 1 "GND" H 9422 6331 50  0000 C CNN
-F 2 "" H 9550 6393 50  0001 C CNN
-F 3 "" H 9550 6393 50  0001 C CNN
-	1    9550 6393
+P 8515 6405
+F 0 "#PWR0109" H 8515 6155 50  0001 C CNN
+F 1 "GND" H 8387 6343 50  0000 C CNN
+F 2 "" H 8515 6405 50  0001 C CNN
+F 3 "" H 8515 6405 50  0001 C CNN
+	1    8515 6405
 	1    0    0    -1
 $EndComp
@@
 L power:GND #PWR0110
 U 1 1 5BDCFC6E
-P 10074 6399
-F 0 "#PWR0110" H 10074 6149 50  0001 C CNN
-F 1 "GND" H 9946 6337 50  0000 C CNN
-F 2 "" H 10074 6399 50  0001 C CNN
-F 3 "" H 10074 6399 50  0001 C CNN
-	1    10074 6399
-	1    0    0    -1
-$EndComp
-$Comp
-L power:GND #PWR0111
-U 1 1 5BDCFCC3
-P 10560 6402
-F 0 "#PWR0111" H 10560 6152 50  0001 C CNN
-F 1 "GND" H 10432 6340 50  0000 C CNN
-F 2 "" H 10560 6402 50  0001 C CNN
-F 3 "" H 10560 6402 50  0001 C CNN
-	1    10560 6402
+P 10070 6385
+F 0 "#PWR0110" H 10070 6135 50  0001 C CNN
+F 1 "GND" H 9942 6323 50  0000 C CNN
+F 2 "" H 10070 6385 50  0001 C CNN
+F 3 "" H 10070 6385 50  0001 C CNN
+	1    10070 6385
 	1    0    0    -1
 $EndComp
@@
 	3279 3754 3279 3982
 $Comp
-L Catwan_Farmer-rescue:74HC4052-electroniccats U5
+L Catwan_Farmer-rescue:74HC4052-electroniccats-Catwan_Farmer-rescue U5
 U 1 1 5C0415EA
 P 8414 5185
@@
 Text Label 1800 2060 2    50   ~ 0
 ADC_BAT
-$Comp
-L Transistor_FET:BSS214NW Q1
-U 1 1 5C6F67E5
-P 8905 6046
-F 0 "Q1" H 9062 6158 50  0000 L CNN
-F 1 "2N7002" H 8544 5805 50  0000 L CNN
-F 2 "Package_TO_SOT_SMD:SOT-23" H 9105 5971 50  0001 L CIN
-F 3 "https://www.infineon.com/dgdl/Infineon-BSS214NW-DS-v02_02-en.pdf?fileId=db3a30431b3e89eb011b695aebc01bde" H 8905 6046 50  0001 L CNN
-	1    8905 6046
-	1    0    0    -1
-$EndComp
-Wire Wire Line
-	8949 5498 10074 5498
-Wire Wire Line
-	9005 6246 9005 6401
-$Comp
-L Transistor_FET:BSS214NW Q2
-U 1 1 5C81EBFF
-P 9450 6038
-F 0 "Q2" H 9606 6146 50  0000 L CNN
-F 1 "2N7002" H 9110 5809 50  0000 L CNN
-F 2 "Package_TO_SOT_SMD:SOT-23" H 9650 5963 50  0001 L CIN
-F 3 "https://www.infineon.com/dgdl/Infineon-BSS214NW-DS-v02_02-en.pdf?fileId=db3a30431b3e89eb011b695aebc01bde" H 9450 6038 50  0001 L CNN
-	1    9450 6038
-	1    0    0    -1
-$EndComp
-Wire Wire Line
-	9550 6238 9550 6393
-Wire Wire Line
-	8813 5746 10341 5746
-Wire Wire Line
-	8910 5646 10227 5646
-$Comp
-L Transistor_FET:BSS214NW Q3
-U 1 1 5C85476C
-P 9974 6048
-F 0 "Q3" H 10121 6166 50  0000 L CNN
-F 1 "2N7002" H 9634 5819 50  0000 L CNN
-F 2 "Package_TO_SOT_SMD:SOT-23" H 10174 5973 50  0001 L CIN
-F 3 "https://www.infineon.com/dgdl/Infineon-BSS214NW-DS-v02_02-en.pdf?fileId=db3a30431b3e89eb011b695aebc01bde" H 9974 6048 50  0001 L CNN
-	1    9974 6048
-	1    0    0    -1
-$EndComp
-$Comp
-L Transistor_FET:BSS214NW Q4
-U 1 1 5C85E227
-P 10460 6049
-F 0 "Q4" H 10642 6173 50  0000 L CNN
-F 1 "2N7002" H 10120 5820 50  0000 L CNN
-F 2 "Package_TO_SOT_SMD:SOT-23" H 10660 5974 50  0001 L CIN
-F 3 "https://www.infineon.com/dgdl/Infineon-BSS214NW-DS-v02_02-en.pdf?fileId=db3a30431b3e89eb011b695aebc01bde" H 10460 6049 50  0001 L CNN
-	1    10460 6049
-	1    0    0    -1
-$EndComp
 Wire Wire Line
 	8814 4885 8940 4885
@@
 	8814 4985 9015 4985
 Wire Wire Line
-	8922 5152 9199 5152
-Wire Wire Line
 	8921 5252 9420 5252
-Wire Wire Line
-	9066 5398 9748 5398
-Wire Wire Line
-	8705 6046 8652 6046
-Wire Wire Line
-	8652 6046 8652 5727
-Wire Wire Line
-	8652 5727 8940 5727
-Wire Wire Line
-	8940 5727 8940 4885
 Connection ~ 8940 4885
 Wire Wire Line
 	8940 4885 10379 4885
-Wire Wire Line
-	9005 5846 9015 5846
-Wire Wire Line
-	9015 5846 9015 4985
 Connection ~ 9015 4985
 Wire Wire Line
 	9015 4985 10379 4985
-Wire Wire Line
-	9250 6038 9199 6038
-Wire Wire Line
-	9199 5152 9199 6038
-Connection ~ 9199 5152
-Wire Wire Line
-	9199 5152 10380 5152
-Wire Wire Line
-	9550 5838 9420 5838
-Wire Wire Line
-	9420 5838 9420 5252
 Connection ~ 9420 5252
 Wire Wire Line
 	9420 5252 10380 5252
-Wire Wire Line
-	9774 6048 9748 6048
-Wire Wire Line
-	9748 6048 9748 5398
-Connection ~ 9748 5398
-Wire Wire Line
-	9748 5398 10384 5398
-Wire Wire Line
-	10074 5498 10074 5848
-Connection ~ 10074 5498
-Wire Wire Line
-	10074 5498 10384 5498
-Wire Wire Line
-	10074 6248 10074 6399
-Wire Wire Line
-	10227 6049 10227 5646
-Wire Wire Line
-	10227 6049 10260 6049
-Connection ~ 10227 5646
-Wire Wire Line
-	10227 5646 10392 5646
-Wire Wire Line
-	10560 5849 10560 5822
-Wire Wire Line
-	10560 5822 10341 5822
-Wire Wire Line
-	10341 5822 10341 5746
-Connection ~ 10341 5746
-Wire Wire Line
-	10341 5746 10392 5746
-Wire Wire Line
-	10560 6249 10560 6402
 Text Label 3200 1860 0    50   ~ 0
 S1
@@
 Text Label 1535 2160 0    50   ~ 0
 SEN_X
+Wire Wire Line
+	8922 5152 9190 5152
+Wire Wire Line
+	9015 5875 9125 5875
+Wire Wire Line
+	9015 4985 9015 5875
+Wire Wire Line
+	8940 5850 8850 5850
+Wire Wire Line
+	8850 5850 8850 5910
+Wire Wire Line
+	8940 4885 8940 5850
+Wire Wire Line
+	9420 5885 9655 5885
+Wire Wire Line
+	9420 5252 9420 5885
+Wire Wire Line
+	9400 5900 9190 5900
+Wire Wire Line
+	9190 5152 9190 5900
+Connection ~ 9190 5152
+Wire Wire Line
+	9190 5152 10380 5152
+Wire Wire Line
+	8949 5498 10180 5498
+Wire Wire Line
+	8910 5646 10249 5646
+Wire Wire Line
+	8813 5746 10334 5746
+Wire Wire Line
+	9066 5398 9910 5398
+Connection ~ 9910 5398
+Wire Wire Line
+	9910 5398 10384 5398
+Connection ~ 10180 5498
+Wire Wire Line
+	10180 5498 10384 5498
+Wire Wire Line
+	10249 5646 10249 5930
+Connection ~ 10249 5646
+Wire Wire Line
+	10249 5646 10392 5646
+Wire Wire Line
+	10334 5746 10334 5897
+Wire Wire Line
+	10334 5897 10700 5897
+Wire Wire Line
+	10700 5897 10700 5925
+Connection ~ 10334 5746
+Wire Wire Line
+	10334 5746 10392 5746
+$Comp
+L power:GND #PWR0111
+U 1 1 5BDCFCC3
+P 10735 6365
+F 0 "#PWR0111" H 10735 6115 50  0001 C CNN
+F 1 "GND" H 10607 6303 50  0000 C CNN
+F 2 "" H 10735 6365 50  0001 C CNN
+F 3 "" H 10735 6365 50  0001 C CNN
+	1    10735 6365
+	1    0    0    -1
+$EndComp
+$Comp
+L Device:D_Zener_x2_ACom_KKA D8
+U 1 1 5D5A9182
+P 8515 6145
+F 0 "D8" H 8515 6361 50  0000 C CNN
+F 1 "AZ23C9V1" H 8515 6270 50  0000 C CNN
+F 2 "" H 8515 6145 50  0001 C CNN
+F 3 "~" H 8515 6145 50  0001 C CNN
+	1    8515 6145
+	1    0    0    -1
+$EndComp
+$Comp
+L Device:D_Zener_x2_ACom_KKA D5
+U 1 1 5D5C7058
+P 9285 6135
+F 0 "D5" H 9285 6351 50  0000 C CNN
+F 1 "AZ23C9V1" H 9285 6260 50  0000 C CNN
+F 2 "" H 9285 6135 50  0001 C CNN
+F 3 "~" H 9285 6135 50  0001 C CNN
+	1    9285 6135
+	1    0    0    -1
+$EndComp
+$Comp
+L Device:D_Zener_x2_ACom_KKA D6
+U 1 1 5D5C7D3F
+P 10070 6135
+F 0 "D6" H 10070 6351 50  0000 C CNN
+F 1 "AZ23C9V1" H 10070 6260 50  0000 C CNN
+F 2 "" H 10070 6135 50  0001 C CNN
+F 3 "~" H 10070 6135 50  0001 C CNN
+	1    10070 6135
+	1    0    0    -1
+$EndComp
+$Comp
+L Device:D_Zener_x2_ACom_KKA D4
+U 1 1 5D5C871F
+P 10735 6100
+F 0 "D4" H 10735 6316 50  0000 C CNN
+F 1 "AZ23C9V1" H 10735 6225 50  0000 C CNN
+F 2 "" H 10735 6100 50  0001 C CNN
+F 3 "~" H 10735 6100 50  0001 C CNN
+	1    10735 6100
+	1    0    0    -1
+$EndComp
+Wire Wire Line
+	10700 5925 11035 5925
+Wire Wire Line
+	11035 5925 11035 6100
+Wire Wire Line
+	10435 6100 10435 5930
+Wire Wire Line
+	10249 5930 10435 5930
+Wire Wire Line
+	10180 6070 10370 6070
+Wire Wire Line
+	10370 6070 10370 6135
+Wire Wire Line
+	10180 5498 10180 6070
+Wire Wire Line
+	9910 6045 9770 6045
+Wire Wire Line
+	9770 6045 9770 6135
+Wire Wire Line
+	9910 5398 9910 6045
+Wire Wire Line
+	9585 6135 9655 6135
+Wire Wire Line
+	9655 6135 9655 5885
+Wire Wire Line
+	9400 5900 9400 6050
+Wire Wire Line
+	9400 6050 8985 6050
+Wire Wire Line
+	8985 6050 8985 6135
+Wire Wire Line
+	8850 5910 8215 5910
+Wire Wire Line
+	8215 5910 8215 6145
+Wire Wire Line
+	9125 5990 8815 5990
+Wire Wire Line
+	8815 5990 8815 6145
+Wire Wire Line
+	9125 5875 9125 5990
+Wire Wire Line
+	8515 6405 8515 6345
+Wire Wire Line
+	9285 6405 9285 6335
+Wire Wire Line
+	10070 6335 10070 6385
+Wire Wire Line
+	10735 6365 10735 6300
 $EndSCHEMATC

Commit message: update led, switch and labels
Parts:
- added D9: LED, LED_SMD:LED_0805_2012Metric_Pad1.15x1.40mm_HandSolder, symbol Device:LED
- added R9: 1K, Resistor_SMD:R_0805_2012Metric_Pad1.15x1.40mm_HandSolder, symbol Device:R
- SW1: symbol Switch:SW_DPST_x2 -> Catwan_Farmer-rescue:SW_DPST_x2-Switch
Connections:
- net SEN_X is gone; now on net SENS_X: U2.6 (PA05)
- net SEN_Y is gone; now on net SENS_Y: U2.8 (PA07)
- net GND: now also R9.2
- net LED: now also D9.2 (A)
- new net: D9.1 (K), R9.1
Other:
- moved on the sheet: D10, R6
Changed lines of the file:
@@
 EESchema Schematic File Version 4
 LIBS:Catwan_Farmer-cache
-EELAYER 29 0
+EELAYER 30 0
 EELAYER END
 $Descr A4 11693 8268
@@
 $EndComp
 $Comp
-L Switch:SW_DPST_x2 SW1
+L Catwan_Farmer-rescue:SW_DPST_x2-Switch SW1
 U 1 1 5BAF7531
 P 1520 1460
@@
 L Device:LED D10
 U 1 1 5BC0A216
-P 10695 1359
-F 0 "D10" V 10733 1242 50  0000 R CNN
-F 1 "LED" V 10642 1242 50  0000 R CNN
-F 2 "LED_SMD:LED_0805_2012Metric_Pad1.15x1.40mm_HandSolder" H 10695 1359 50  0001 C CNN
-F 3 "~" H 10695 1359 50  0001 C CNN
-	1    10695 1359
+P 10710 1379
+F 0 "D10" V 10748 1262 50  0000 R CNN
+F 1 "LED" V 10657 1262 50  0000 R CNN
+F 2 "LED_SMD:LED_0805_2012Metric_Pad1.15x1.40mm_HandSolder" H 10710 1379 50  0001 C CNN
+F 3 "~" H 10710 1379 50  0001 C CNN
+	1    10710 1379
 	0    -1   -1   0
 $EndComp
@@
 L Device:R R6
 U 1 1 5BCA3EA8
-P 10695 1785
-F 0 "R6" H 10765 1831 50  0000 L CNN
-F 1 "1K" H 10765 1740 50  0000 L CNN
-F 2 "Resistor_SMD:R_0805_2012Metric_Pad1.15x1.40mm_HandSolder" V 10625 1785 50  0001 C CNN
-F 3 "~" H 10695 1785 50  0001 C CNN
-	1    10695 1785
-	1    0    0    -1
-$EndComp
-Wire Wire Line
-	10695 1635 10695 1509
+P 10710 1805
+F 0 "R6" H 10780 1851 50  0000 L CNN
+F 1 "1K" H 10780 1760 50  0000 L CNN
+F 2 "Resistor_SMD:R_0805_2012Metric_Pad1.15x1.40mm_HandSolder" V 10640 1805 50  0001 C CNN
+F 3 "~" H 10710 1805 50  0001 C CNN
+	1    10710 1805
+	1    0    0    -1
+$EndComp
+Wire Wire Line
+	10710 1655 10710 1529
 $Comp
 L power:GND #PWR025
 U 1 1 5BCA951A
-P 10695 2005
-F 0 "#PWR025" H 10695 1755 50  0001 C CNN
-F 1 "GND" H 10700 1832 50  0000 C CNN
-F 2 "" H 10695 2005 50  0001 C CNN
-F 3 "" H 10695 2005 50  0001 C CNN
-	1    10695 2005
+P 10710 2025
+F 0 "#PWR025" H 10710 1775 50  0001 C CNN
+F 1 "GND" H 10715 1852 50  0000 C CNN
+F 2 "" H 10710 2025 50  0001 C CNN
+F 3 "" H 10710 2025 50  0001 C CNN
+	1    10710 2025
 	1    0    0    -1
 $EndComp
@@
 L power:+3.3V #PWR024
 U 1 1 5BCA956B
-P 10695 1059
-F 0 "#PWR024" H 10695 909 50  0001 C CNN
-F 1 "+3.3V" H 10710 1232 50  0000 C CNN
-F 2 "" H 10695 1059 50  0001 C CNN
-F 3 "" H 10695 1059 50  0001 C CNN
-	1    10695 1059
-	1    0    0    -1
-$EndComp
-Wire Wire Line
-	10695 1209 10695 1059
-Wire Wire Line
-	10695 1935 10695 2005
+P 10710 1079
+F 0 "#PWR024" H 10710 929 50  0001 C CNN
+F 1 "+3.3V" H 10725 1252 50  0000 C CNN
+F 2 "" H 10710 1079 50  0001 C CNN
+F 3 "" H 10710 1079 50  0001 C CNN
+	1    10710 1079
+	1    0    0    -1
+$EndComp
+Wire Wire Line
+	10710 1229 10710 1079
+Wire Wire Line
+	10710 1955 10710 2025
 $Comp
 L power:GND #PWR020
@@
 LED
 Text Label 1515 2360 0    50   ~ 0
-SEN_Y
+SENS_Y
 Text Label 1535 2160 0    50   ~ 0
-SEN_X
+SENS_X
 Wire Wire Line
 	8922 5152 9190 5152
@@
 Wire Wire Line
 	10735 6365 10735 6300
+$Comp
+L Device:LED D9
+U 1 1 5E206ABC
+P 6600 1289
+F 0 "D9" V 6638 1172 50  0000 R CNN
+F 1 "LED" V 6547 1172 50  0000 R CNN
+F 2 "LED_SMD:LED_0805_2012Metric_Pad1.15x1.40mm_HandSolder" H 6600 1289 50  0001 C CNN
+F 3 "~" H 6600 1289 50  0001 C CNN
+	1    6600 1289
+	0    -1   -1   0
+$EndComp
+$Comp
+L Device:R R9
+U 1 1 5E206AC2
+P 6600 1715
+F 0 "R9" H 6670 1761 50  0000 L CNN
+F 1 "1K" H 6670 1670 50  0000 L CNN
+F 2 "Resistor_SMD:R_0805_2012Metric_Pad1.15x1.40mm_HandSolder" V 6530 1715 50  0001 C CNN
+F 3 "~" H 6600 1715 50  0001 C CNN
+	1    6600 1715
+	1    0    0    -1
+$EndComp
+Wire Wire Line
+	6600 1565 6600 1439
+$Comp
+L power:GND #PWR0119
+U 1 1 5E206AC9
+P 6600 1935
+F 0 "#PWR0119" H 6600 1685 50  0001 C CNN
+F 1 "GND" H 6605 1762 50  0000 C CNN
+F 2 "" H 6600 1935 50  0001 C CNN
+F 3 "" H 6600 1935 50  0001 C CNN
+	1    6600 1935
+	1    0    0    -1
+$EndComp
+Wire Wire Line
+	6600 1139 6600 989
+Wire Wire Line
+	6600 1865 6600 1935
+Text Label 6600 990  0    50   ~ 0
+LED
 $EndSCHEMATC

Commit message: Change sens_y analog pin
Parts:
- SW1: symbol Catwan_Farmer-rescue:SW_DPST_x2-Switch -> Catwan_Farmer-rescue:SW_DPST_x2-Switch-Catwan_Farmer-rescue
- U2: symbol Catwan_Farmer-rescue:ATSAMD21E18A-MU-electroniccats-Catwan_sensorwater-rescue-Catwan_sensorwater-rescue-Catwan_sensorwater-rescue-Catwan_sensorwater-rescue-Catwan_sensorwater-rescue-Catwan_Farmer-rescue-Catwan_Farmer-rescue -> Catwan_Farmer-rescue:ATSAMD21E18A-MU-electroniccats-Catwan_sensorwater-rescue-Catwan_sensorwater-rescue-Catwan_sensorwater-rescue-Catwan_sensorwater-rescue-Catwan_sensorwater-rescue-Catwan_Farmer-rescue-Catwan_Farmer-rescue-Catwan_Farmer-rescue
- U3: symbol Catwan_Farmer-rescue:RFM95W-868S2-RF_AM_FM -> Catwan_Farmer-rescue:RFM95W-868S2-RF_AM_FM-Catwan_Farmer-rescue
- U5: symbol Catwan_Farmer-rescue:74HC4052-electroniccats-Catwan_Farmer-rescue -> Catwan_Farmer-rescue:74HC4052-electroniccats-Catwan_Farmer-rescue-Catwan_Farmer-rescue
Connections:
- net SENS_Y: now also U2.7 (PA06); no longer U2.8 (PA07)
Changed lines of the file:
@@
 $EndComp
 $Comp
-L Catwan_Farmer-rescue:SW_DPST_x2-Switch SW1
+L Catwan_Farmer-rescue:SW_DPST_x2-Switch-Catwan_Farmer-rescue SW1
 U 1 1 5BAF7531
 P 1520 1460
@@
 	2166 6480 2066 6480
 $Comp
-L Catwan_Farmer-rescue:RFM95W-868S2-RF_AM_FM U3
+L Catwan_Farmer-rescue:RFM95W-868S2-RF_AM_FM-Catwan_Farmer-rescue U3
 U 1 1 5BAF85CF
 P 2066 5762
@@
 	3279 3754 3279 3982
 $Comp
-L Catwan_Farmer-rescue:74HC4052-electroniccats-Catwan_Farmer-rescue U5
+L Catwan_Farmer-rescue:74HC4052-electroniccats-Catwan_Farmer-rescue-Catwan_Farmer-rescue U5
 U 1 1 5C0415EA
 P 8414 5185
@@
 $EndComp
 $Comp
-L Catwan_Farmer-rescue:ATSAMD21E18A-MU-electroniccats-Catwan_sensorwater-rescue-Catwan_sensorwater-rescue-Catwan_sensorwater-rescue-Catwan_sensorwater-rescue-Catwan_sensorwater-rescue-Catwan_Farmer-rescue-Catwan_Farmer-rescue U2
+L Catwan_Farmer-rescue:ATSAMD21E18A-MU-electroniccats-Catwan_sensorwater-rescue-Catwan_sensorwater-rescue-Catwan_sensorwater-rescue-Catwan_sensorwater-rescue-Catwan_sensorwater-rescue-Catwan_Farmer-rescue-Catwan_Farmer-rescue-Catwan_Farmer-rescue U2
 U 1 1 5BAD6569
 P 2500 2160
@@
 Wire Wire Line
 	1720 1460 1800 1460
-NoConn ~ 1800 2260
+NoConn ~ 1800 2362
 Wire Wire Line
 	5020 7220 5020 7120
@@
 	770  2290 970  2290
 Wire Wire Line
-	1800 2460 1515 2460
-Wire Wire Line
-	1800 2360 1515 2360
-Wire Wire Line
 	1800 2160 1535 2160
-Text Label 1515 2460 0    50   ~ 0
+Text Label 1600 2460 0    50   ~ 0
 LED
-Text Label 1515 2360 0    50   ~ 0
+Text Label 1530 2260 0    50   ~ 0
 SENS_Y
 Text Label 1535 2160 0    50   ~ 0
@@
 Text Label 6600 990  0    50   ~ 0
 LED
+Wire Wire Line
+	1800 2460 1600 2460
+Wire Wire Line
+	1530 2260 1800 2260
 $EndSCHEMATC
