File: Hardware/Catwan_Farmer.sch (KiCad schematic (older format))
At the start: 49 parts, among them J1 SENSOR 1, J10 VSP, J2 SENSOR 2, J3 SENSOR 3, J4 BATT, J5 USB_B, J6 Conn_01x04, J7 DHT22, J9 SENSOR 4, SW1 SW_Push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

Commit message: Update V1.0
Parts:
- D10: value LED -> ON
- J6: value Conn_01x04 -> SWD
- SW1: value SW_Push -> RST
- U3: symbol Catwan_Farmer-rescue:ATSAMD21E18A-MU-Electronic_Cats-Catwan_Farmer-rescue -> Catwan_Farmer-rescue:ATSAMD21E18A-MU-Electronic_Cats-Catwan_Farmer-rescue-Catwan_Farmer-rescue
- U5: symbol Catwan_Farmer-rescue:74HC4052-Electronic_Cats-Catwan_Farmer-rescue -> Catwan_Farmer-rescue:74HC4052-Electronic_Cats-Catwan_Farmer-rescue-Catwan_Farmer-rescue
Changed lines of the file:
@@
 EESchema Schematic File Version 4
-LIBS:Catwan_Farmer-cache
 EELAYER 30 0
 EELAYER END
@@
 Sheet 1 1
 Title "CatWAN"
-Date "2019-05-27"
-Rev "0.5"
+Date "2020-06-15"
+Rev "1.0"
 Comp "Electronic Cats"
 Comment1 "Montserrat Figueroa"
@@
 Text Label 3200 1960 0    50   ~ 0
 S0
-Text Label 989  3279 3    50   ~ 0
+Text Label 889  3279 3    50   ~ 0
 SWCLK
 Text Label 1296 6057 2    50   ~ 0
@@
 P 10710 1379
 F 0 "D10" V 10748 1262 50  0000 R CNN
-F 1 "LED" V 10657 1262 50  0000 R CNN
+F 1 "ON" V 10657 1262 50  0000 R CNN
 F 2 "LED_SMD:LED_0805_2012Metric_Pad1.15x1.40mm_HandSolder" H 10710 1379 50  0001 C CNN
 F 3 "~" H 10710 1379 50  0001 C CNN
@@
 P 889 3079
 F 0 "J6" V 855 2791 50  0000 R CNN
-F 1 "Conn_01x04" V 764 2791 50  0000 R CNN
+F 1 "SWD" V 764 2791 50  0000 R CNN
 F 2 "Connector_PinHeader_2.54mm:PinHeader_1x04_P2.54mm_Vertical" H 889 3079 50  0001 C CNN
 F 3 "~" H 889 3079 50  0001 C CNN
@@
 	0    -1   -1   0
 $EndComp
-Text Label 889  3279 3    50   ~ 0
+Text Label 989  3279 3    50   ~ 0
 SWDIO
 Wire Wire Line
@@
 U 1 1 5C6E769E
 P 870 2020
-F 0 "Y1" H 1035 2015 50  0000 C CNN
-F 1 "32.768Khz" H 870 2154 50  0000 C CNN
+F 0 "Y1" H 1035 2085 50  0000 C CNN
+F 1 "32.768Khz" H 1190 2015 50  0000 C CNN
 F 2 "Crystal:Crystal_SMD_MicroCrystal_CC7V-T1A-2Pin_3.2x1.5mm_HandSoldering" H 870 2020 50  0001 C CNN
 F 3 "~" H 870 2020 50  0001 C CNN
@@
 F 4 "" H 8895 4255 50  0001 C CNN "manf#"
 	1    8895 4255
-	1    0    0    -1
+	-1   0    0    -1
 $EndComp
 $Comp
@@
 P 1520 1460
 F 0 "SW1" H 1520 1745 50  0000 C CNN
-F 1 "SW_Push" H 1520 1654 50  0000 C CNN
+F 1 "RST" H 1520 1654 50  0000 C CNN
 F 2 "Button_Switch_SMD:SW_SPST_SKQG_WithStem" H 1520 1660 50  0001 C CNN
 F 3 "~" H 1520 1660 50  0001 C CNN
@@
 	6975 4725 6965 4725
 $Comp
-L Catwan_Farmer-rescue:ATSAMD21E18A-MU-Electronic_Cats-Catwan_Farmer-rescue U3
+L Catwan_Farmer-rescue:ATSAMD21E18A-MU-Electronic_Cats-Catwan_Farmer-rescue-Catwan_Farmer-rescue U3
 U 1 1 5E7C2C42
 P 2500 2160
@@
 $EndComp
 $Comp
-L Catwan_Farmer-rescue:74HC4052-Electronic_Cats-Catwan_Farmer-rescue U5
+L Catwan_Farmer-rescue:74HC4052-Electronic_Cats-Catwan_Farmer-rescue-Catwan_Farmer-rescue U5
 U 1 1 5E7C5328
 P 6390 3310

Commit message: Manf#
Parts:
- C1, C10, C11, C13, C2, C3, C4, C5, C6, C7, C8, D10, D7, D9, R3, R4, R5, R6, R7, R9, SW1, U2: manf# (none) -> -
- D1, D2, D3: manf# (none) -> NRVB120VLSFT1G
- D4, D6, D8: manf# (none) -> AZ23C2V7
- J5: manf# (none) -> C46394
- J7: manf# (none) -> DHT22 AM2302
- R1, R2: manf# (none) -> CRCW0805J-4.7K-E3
- R8: manf# (none) -> CRGP0805F47K
- U1: manf# (none) -> AP2114H-3.3TRG1
- U3: symbol Catwan_Farmer-rescue:ATSAMD21E18A-MU-Electronic_Cats-Catwan_Farmer-rescue-Catwan_Farmer-rescue -> Catwan_Farmer-rescue:ATSAMD21E18A-MU-Electronic_Cats-Catwan_Farmer-rescue-Catwan_Farmer-rescue-Catwan_Farmer-rescue; manf# (none) -> ATSAMD21E18A-AU
- U4: manf# (none) -> MCP73831-3-OT
- U5: symbol Catwan_Farmer-rescue:74HC4052-Electronic_Cats-Catwan_Farmer-rescue-Catwan_Farmer-rescue -> Catwan_Farmer-rescue:74HC4052-Electronic_Cats-Catwan_Farmer-rescue-Catwan_Farmer-rescue-Catwan_Farmer-rescue; manf# (none) -> 74HC4052D,653
- Y1: manf# (none) -> LFXTAL009678Reel
Changed lines of the file:
@@
 EESchema Schematic File Version 4
+LIBS:Catwan_Farmer-cache
 EELAYER 30 0
 EELAYER END
@@
 F 2 "Package_TO_SOT_SMD:SOT-223-3_TabPin2" H 9160 1735 50  0001 C CIN
 F 3 "https://www.diodes.com/assets/Datasheets/AP2127.pdf" H 9160 1510 50  0001 C CNN
+F 4 "AP2114H-3.3TRG1" H 9160 1510 50  0001 C CNN "manf#"
 	1    9160 1510
 	1    0    0    -1
@@
 F 2 "Capacitor_SMD:C_0805_2012Metric_Pad1.15x1.40mm_HandSolder" H 9688 1560 50  0001 C CNN
 F 3 "~" H 9650 1710 50  0001 C CNN
+F 4 "-" H 9650 1710 50  0001 C CNN "manf#"
 	1    9650 1710
 	1    0    0    -1
@@
 F 2 "Capacitor_SMD:C_0805_2012Metric_Pad1.15x1.40mm_HandSolder" H 10098 1560 50  0001 C CNN
 F 3 "~" H 10060 1710 50  0001 C CNN
+F 4 "-" H 10060 1710 50  0001 C CNN "manf#"
 	1    10060 1710
 	1    0    0    -1
@@
 F 2 "Capacitor_SMD:C_0805_2012Metric_Pad1.15x1.40mm_HandSolder" H 652 5931 50  0001 C CNN
 F 3 "~" H 614 6081 50  0001 C CNN
+F 4 "-" H 614 6081 50  0001 C CNN "manf#"
 	1    614  6081
 	1    0    0    -1
@@
 F 2 "Connectors electroniccats:U254051N4BH806" H 5459 1454 50  0001 C CNN
 F 3 " ~" H 5459 1454 50  0001 C CNN
+F 4 "	C46394" H 5309 1504 50  0001 C CNN "manf#"
 	1    5309 1504
 	1    0    0    -1
@@
 F 2 "Resistor_SMD:R_0805_2012Metric_Pad1.15x1.40mm_HandSolder" V 5635 3490 50  0001 C CNN
 F 3 "~" H 5705 3490 50  0001 C CNN
+F 4 "CRCW0805J-4.7K-E3" H 5705 3490 50  0001 C CNN "manf#"
 	1    5705 3490
 	1    0    0    -1
@@
 F 2 "LED_SMD:LED_0805_2012Metric_Pad1.15x1.40mm_HandSolder" H 10710 1379 50  0001 C CNN
 F 3 "~" H 10710 1379 50  0001 C CNN
+F 4 "-" H 10710 1379 50  0001 C CNN "manf#"
 	1    10710 1379
 	0    -1   -1   0
@@
 F 2 "Resistor_SMD:R_0805_2012Metric_Pad1.15x1.40mm_HandSolder" V 4115 6775 50  0001 C CNN
 F 3 "~" H 4185 6775 50  0001 C CNN
+F 4 "-" H 4185 6775 50  0001 C CNN "manf#"
 	1    4185 6775
 	-1   0    0    1
@@
 F 2 "Resistor_SMD:R_0805_2012Metric_Pad1.15x1.40mm_HandSolder" V 10640 1805 50  0001 C CNN
 F 3 "~" H 10710 1805 50  0001 C CNN
+F 4 "-" H 10710 1805 50  0001 C CNN "manf#"
 	1    10710 1805
 	1    0    0    -1
@@
 F 2 "Capacitor_SMD:C_0805_2012Metric_Pad1.15x1.40mm_HandSolder" H 4186 2846 50  0001 C CNN
 F 3 "~" H 4148 2996 50  0001 C CNN
+F 4 "-" H 4148 2996 50  0001 C CNN "manf#"
 	1    4148 2996
 	1    0    0    -1
@@
 F 2 "Capacitor_SMD:C_0805_2012Metric_Pad1.15x1.40mm_HandSolder" H 3588 1440 50  0001 C CNN
 F 3 "~" H 3550 1590 50  0001 C CNN
+F 4 "-" H 3550 1590 50  0001 C CNN "manf#"
 	1    3550 1590
 	1    0    0    -1
@@
 F 2 "Diode_SMD:D_SOD-123" H 8380 1260 50  0001 C CNN
 F 3 "~" H 8380 1260 50  0001 C CNN
+F 4 "NRVB120VLSFT1G" H 8380 1260 50  0001 C CNN "manf#"
 	1    8380 1260
 	0    -1   -1   0
@@
 F 2 "Capacitor_SMD:C_0805_2012Metric_Pad1.15x1.40mm_HandSolder" H 8418 1570 50  0001 C CNN
 F 3 "~" H 8380 1720 50  0001 C CNN
+F 4 "-" H 8380 1720 50  0001 C CNN "manf#"
 	1    8380 1720
 	1    0    0    -1
@@
 F 2 "Package_TO_SOT_SMD:SOT-23-5" H 4655 6065 50  0001 L CIN
 F 3 "http://ww1.microchip.com/downloads/en/DeviceDoc/20001984g.pdf" H 4455 6265 50  0001 C CNN
+F 4 "MCP73831-3-OT" H 4605 6315 50  0001 C CNN "manf#"
 	1    4605 6315
 	1    0    0    -1
@@
 F 2 "LED_SMD:LED_0805_2012Metric_Pad1.15x1.40mm_HandSolder" H 5675 5915 50  0001 C CNN
 F 3 "~" H 5675 5915 50  0001 C CNN
+F 4 "-" H 5675 5915 50  0001 C CNN "manf#"
 	1    5675 5915
 	0    -1   -1   0
@@
 F 2 "Resistor_SMD:R_0805_2012Metric_Pad1.15x1.40mm_HandSolder" V 5605 6265 50  0001 C CNN
 F 3 "~" H 5675 6265 50  0001 C CNN
+F 4 "-" H 5675 6265 50  0001 C CNN "manf#"
 	1    5675 6265
 	-1   0    0    1
@@
 F 2 "Capacitor_SMD:C_0805_2012Metric_Pad1.15x1.40mm_HandSolder" H 5173 6895 50  0001 C CNN
 F 3 "~" H 5135 7045 50  0001 C CNN
+F 4 "-" H 5135 7045 50  0001 C CNN "manf#"
 	1    5135 7045
 	-1   0    0    1
@@
 F 2 "Capacitor_SMD:C_0805_2012Metric_Pad1.15x1.40mm_HandSolder" H 3468 910 50  0001 C CNN
 F 3 "~" H 3430 1060 50  0001 C CNN
+F 4 "-" H 3430 1060 50  0001 C CNN "manf#"
 	1    3430 1060
 	0    1    1    0
@@
 F 2 "Diode_SMD:D_SOD-123" H 5824 1100 50  0001 C CNN
 F 3 "~" H 5824 1100 50  0001 C CNN
+F 4 "NRVB120VLSFT1G" H 5824 1100 50  0001 C CNN "manf#"
 	1    5824 1100
 	0    1    1    0
@@
 F 2 "Diode_SMD:D_SOD-123" H 4295 5545 50  0001 C CNN
 F 3 "~" H 4295 5545 50  0001 C CNN
+F 4 "NRVB120VLSFT1G" H 4295 5545 50  0001 C CNN "manf#"
 	1    4295 5545
 	-1   0    0    1
@@
 F 2 "Capacitor_SMD:C_0805_2012Metric_Pad1.15x1.40mm_HandSolder" H 3927 6099 50  0001 C CNN
 F 3 "~" H 3889 6249 50  0001 C CNN
+F 4 "-" H 3889 6249 50  0001 C CNN "manf#"
 	1    3889 6249
 	1    0    0    -1
@@
 F 2 "Crystal:Crystal_SMD_MicroCrystal_CC7V-T1A-2Pin_3.2x1.5mm_HandSoldering" H 870 2020 50  0001 C CNN
 F 3 "~" H 870 2020 50  0001 C CNN
+F 4 "LFXTAL009678Reel" H 870 2020 50  0001 C CNN "manf#"
 	1    870  2020
 	1    0    0    -1
@@
 F 2 "Resistor_SMD:R_0805_2012Metric_Pad1.15x1.40mm_HandSolder" H 7410 1130 50  0001 C CNN
 F 3 "~" H 7410 1130 50  0001 C CNN
+F 4 "-" H 7410 1130 50  0001 C CNN "manf#"
 	1    7410 1130
 	1    0    0    -1
@@
 F 2 "Resistor_SMD:R_0805_2012Metric_Pad1.15x1.40mm_HandSolder" H 7410 1390 50  0001 C CNN
 F 3 "~" H 7410 1390 50  0001 C CNN
+F 4 "-" H 7410 1390 50  0001 C CNN "manf#"
 	1    7410 1390
 	1    0    0    -1
@@
 F 2 "Package_TO_SOT_SMD:SOT-23" H 7225 4255 50  0001 C CNN
 F 3 "~" H 7225 4255 50  0001 C CNN
+F 4 "AZ23C2V7" H 7225 4255 50  0001 C CNN "manf#"
 	1    7225 4255
 	1    0    0    -1
@@
 F 2 "Package_TO_SOT_SMD:SOT-23" H 8895 4255 50  0001 C CNN
 F 3 "~" H 8895 4255 50  0001 C CNN
-F 4 "" H 8895 4255 50  0001 C CNN "manf#"
+F 4 "AZ23C2V7" H 8895 4255 50  0001 C CNN "manf#"
 	1    8895 4255
 	-1   0    0    -1
@@
 F 2 "Package_TO_SOT_SMD:SOT-23" H 9640 4250 50  0001 C CNN
 F 3 "~" H 9640 4250 50  0001 C CNN
+F 4 "AZ23C2V7" H 9640 4250 50  0001 C CNN "manf#"
 	1    9640 4250
 	1    0    0    -1
@@
 F 2 "Resistor_SMD:R_0805_2012Metric_Pad1.15x1.40mm_HandSolder" V 6530 1715 50  0001 C CNN
 F 3 "~" H 6600 1715 50  0001 C CNN
+F 4 "-" H 6600 1715 50  0001 C CNN "manf#"
 	1    6600 1715
 	1    0    0    -1
@@
 F 2 "RF_Module:HOPERF_RFM9XW_SMD" H -1504 7807 50  0001 C CNN
 F 3 "https://www.hoperf.com/data/upload/portal/20181127/5bfcbea20e9ef.pdf" H -1504 7807 50  0001 C CNN
+F 4 "-" H 1796 6157 50  0001 C CNN "manf#"
 	1    1796 6157
 	1    0    0    -1
@@
 F 2 "Resistor_SMD:R_0805_2012Metric_Pad1.15x1.40mm_HandSolder" V 5385 3490 50  0001 C CNN
 F 3 "~" H 5455 3490 50  0001 C CNN
+F 4 "CRCW0805J-4.7K-E3" H 5455 3490 50  0001 C CNN "manf#"
 	1    5455 3490
 	1    0    0    -1
@@
 F 2 "Capacitor_SMD:C_0805_2012Metric_Pad1.15x1.40mm_HandSolder" H 9603 5710 50  0001 C CNN
 F 3 "~" H 9565 5860 50  0001 C CNN
+F 4 "-" H 9565 5860 50  0001 C CNN "manf#"
 	1    9565 5860
 	1    0    0    -1
@@
 F 2 "Resistor_SMD:R_0805_2012Metric_Pad1.15x1.40mm_HandSolder" H 9965 5850 50  0001 C CNN
 F 3 "~" H 9965 5850 50  0001 C CNN
+F 4 "CRGP0805F47K" H 9965 5850 50  0001 C CNN "manf#"
 	1    9965 5850
 	1    0    0    -1
@@
 F 2 "Connector_PinHeader_2.54mm:PinHeader_1x04_P2.54mm_Vertical" H 10345 5750 50  0001 C CNN
 F 3 "~" H 10345 5750 50  0001 C CNN
+F 4 "DHT22 AM2302" H 10345 5750 50  0001 C CNN "manf#"
 	1    10345 5750
 	1    0    0    -1
@@
 F 2 "Button_Switch_SMD:SW_SPST_SKQG_WithStem" H 1520 1660 50  0001 C CNN
 F 3 "~" H 1520 1660 50  0001 C CNN
+F 4 "-" H 1520 1460 50  0001 C CNN "manf#"
 	1    1520 1460
 	1    0    0    -1
@@
 	6975 4725 6965 4725
 $Comp
-L Catwan_Farmer-rescue:ATSAMD21E18A-MU-Electronic_Cats-Catwan_Farmer-rescue-Catwan_Farmer-rescue U3
+L Catwan_Farmer-rescue:ATSAMD21E18A-MU-Electronic_Cats-Catwan_Farmer-rescue-Catwan_Farmer-rescue-Catwan_Farmer-rescue U3
 U 1 1 5E7C2C42
 P 2500 2160
@@
 F 2 "Package_QFP:TQFP-32_7x7mm_P0.8mm" H 2500 2160 50  0001 L BNN
 F 3 "SAMD21E Series 256 KB Flash 32 KB SRAM 48 MHz 32-Bit Microcontroller - QFN-32" H 2500 2160 50  0001 L BNN
+F 4 "ATSAMD21E18A-AU" H 2500 2160 50  0001 C CNN "manf#"
 	1    2500 2160
 	1    0    0    -1
 $EndComp
 $Comp
-L Catwan_Farmer-rescue:74HC4052-Electronic_Cats-Catwan_Farmer-rescue-Catwan_Farmer-rescue U5
+L Catwan_Farmer-rescue:74HC4052-Electronic_Cats-Catwan_Farmer-rescue-Catwan_Farmer-rescue-Catwan_Farmer-rescue U5
 U 1 1 5E7C5328
 P 6390 3310
@@
 F 2 "Package_SO:SOIC-16_3.9x9.9mm_P1.27mm" H 6390 3310 50  0001 C CNN
 F 3 "Sig/Phil 74hc4052d Smd 50/Tube" H 6390 3310 50  0001 L BNN
+F 4 "74HC4052D,653" H 6390 3310 50  0001 C CNN "manf#"
 	1    6390 3310
 	1    0    0    -1
@@
 F 2 "LED_SMD:LED_0805_2012Metric_Pad1.15x1.40mm_HandSolder" H 6600 1290 50  0001 C CNN
 F 3 "~" H 6600 1290 50  0001 C CNN
+F 4 "-" H 6600 1290 50  0001 C CNN "manf#"
 	1    6600 1290
 	0    -1   -1   0
@@
 F 2 "Capacitor_SMD:C_0805_2012Metric_Pad1.15x1.40mm_HandSolder" H 4008 1440 50  0001 C CNN
 F 3 "~" H 3970 1590 50  0001 C CNN
+F 4 "-" H 3970 1590 50  0001 C CNN "manf#"
 	1    3970 1590
 	1    0    0    -1

Commit message: fix error pinout sensors
Parts:
- U3: symbol Catwan_Farmer-rescue:ATSAMD21E18A-MU-Electronic_Cats-Catwan_Farmer-rescue-Catwan_Farmer-rescue-Catwan_Farmer-rescue -> Catwan_Farmer-rescue:ATSAMD21E18A-MU-Electronic_Cats-Catwan_Farmer-rescue-Catwan_Farmer-rescue-Catwan_Farmer-rescue-Cat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
- U5: symbol Catwan_Farmer-rescue:74HC4052-Electronic_Cats-Catwan_Farmer-rescue-Catwan_Farmer-rescue-Catwan_Farmer-rescue -> Catwan_Farmer-rescue:74HC4052-Electronic_Cats-Catwan_Farmer-rescue-Catwan_Farmer-rescue-Catwan_Farmer-rescue-Catwan_Far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
Connections:
- net SENS_X1: now reaches J1.1 (Pin_1), U5.12 (X0)
- net SENS_X1: now also D8.2 (K); no longer D8.1 (K)
- net SENS_Y4: now reaches J9.2 (Pin_2), U5.4 (Y3)
- net SENS_Y4: now also D4.1 (K); no longer D4.2 (K)
- new net SENS_X2: D5.2 (K), J2.1 (Pin_1), U5.14 (X1)
- new net SENS_X3: D6.1 (K), J3.1 (Pin_1), U5.15 (X2)
- new net SENS_X4: D4.2 (K), J9.1 (Pin_1), U5.11 (X3)
- new net SENS_Y1: D8.1 (K), J1.2 (Pin_2), U5.1 (Y0)
- new net SENS_Y2: D5.1 (K), J2.2 (Pin_2), U5.5 (Y1)
- new net SENS_Y3: D6.2 (K), J3.2 (Pin_2), U5.2 (Y2)
Other:
- moved on the sheet: D4, D6, D8
Changed lines of the file:
@@
 EESchema Schematic File Version 4
-LIBS:Catwan_Farmer-cache
 EELAYER 30 0
 EELAYER END
@@
 L power:GND #PWR0109
 U 1 1 5BDCFBA0
-P 7225 4515
-F 0 "#PWR0109" H 7225 4265 50  0001 C CNN
-F 1 "GND" H 7097 4453 50  0000 C CNN
-F 2 "" H 7225 4515 50  0001 C CNN
-F 3 "" H 7225 4515 50  0001 C CNN
-	1    7225 4515
+P 6705 4560
+F 0 "#PWR0109" H 6705 4310 50  0001 C CNN
+F 1 "GND" H 6577 4498 50  0000 C CNN
+F 2 "" H 6705 4560 50  0001 C CNN
+F 3 "" H 6705 4560 50  0001 C CNN
+	1    6705 4560
 	1    0    0    -1
 $EndComp
@@
 L power:GND #PWR0110
 U 1 1 5BDCFC6E
-P 8895 4505
-F 0 "#PWR0110" H 8895 4255 50  0001 C CNN
-F 1 "GND" H 8767 4443 50  0000 C CNN
-F 2 "" H 8895 4505 50  0001 C CNN
-F 3 "" H 8895 4505 50  0001 C CNN
-	1    8895 4505
+P 9425 4515
+F 0 "#PWR0110" H 9425 4265 50  0001 C CNN
+F 1 "GND" H 9297 4453 50  0000 C CNN
+F 2 "" H 9425 4515 50  0001 C CNN
+F 3 "" H 9425 4515 50  0001 C CNN
+	1    9425 4515
 	1    0    0    -1
 $EndComp
@@
 L power:GND #PWR0111
 U 1 1 5BDCFCC3
-P 9640 4515
-F 0 "#PWR0111" H 9640 4265 50  0001 C CNN
-F 1 "GND" H 9512 4453 50  0000 C CNN
-F 2 "" H 9640 4515 50  0001 C CNN
-F 3 "" H 9640 4515 50  0001 C CNN
-	1    9640 4515
+P 10570 4520
+F 0 "#PWR0111" H 10570 4270 50  0001 C CNN
+F 1 "GND" H 10442 4458 50  0000 C CNN
+F 2 "" H 10570 4520 50  0001 C CNN
+F 3 "" H 10570 4520 50  0001 C CNN
+	1    10570 4520
 	1    0    0    -1
 $EndComp
@@
 L Device:D_Zener_x2_ACom_KKA D8
 U 1 1 5D5A9182
-P 7225 4255
-F 0 "D8" H 7225 4471 50  0000 C CNN
-F 1 "AZ23C9V1" H 7225 4380 50  0000 C CNN
-F 2 "Package_TO_SOT_SMD:SOT-23" H 7225 4255 50  0001 C CNN
-F 3 "~" H 7225 4255 50  0001 C CNN
-F 4 "AZ23C2V7" H 7225 4255 50  0001 C CNN "manf#"
-	1    7225 4255
+P 6705 4300
+F 0 "D8" H 6705 4516 50  0000 C CNN
+F 1 "AZ23C9V1" H 6705 4425 50  0000 C CNN
+F 2 "Package_TO_SOT_SMD:SOT-23" H 6705 4300 50  0001 C CNN
+F 3 "~" H 6705 4300 50  0001 C CNN
+F 4 "AZ23C2V7" H 6705 4300 50  0001 C CNN "manf#"
+	1    6705 4300
 	1    0    0    -1
 $EndComp
@@
 L Device:D_Zener_x2_ACom_KKA D6
 U 1 1 5D5C7D3F
-P 8895 4255
-F 0 "D6" H 8895 4471 50  0000 C CNN
-F 1 "AZ23C9V1" H 8895 4380 50  0000 C CNN
-F 2 "Package_TO_SOT_SMD:SOT-23" H 8895 4255 50  0001 C CNN
-F 3 "~" H 8895 4255 50  0001 C CNN
-F 4 "AZ23C2V7" H 8895 4255 50  0001 C CNN "manf#"
-	1    8895 4255
+P 9425 4265
+F 0 "D6" H 9425 4481 50  0000 C CNN
+F 1 "AZ23C9V1" H 9425 4390 50  0000 C CNN
+F 2 "Package_TO_SOT_SMD:SOT-23" H 9425 4265 50  0001 C CNN
+F 3 "~" H 9425 4265 50  0001 C CNN
+F 4 "AZ23C2V7" H 9425 4265 50  0001 C CNN "manf#"
+	1    9425 4265
 	-1   0    0    -1
 $EndComp
@@
 L Device:D_Zener_x2_ACom_KKA D4
 U 1 1 5D5C871F
-P 9640 4250
-F 0 "D4" H 9640 4466 50  0000 C CNN
-F 1 "AZ23C9V1" H 9640 4375 50  0000 C CNN
-F 2 "Package_TO_SOT_SMD:SOT-23" H 9640 4250 50  0001 C CNN
-F 3 "~" H 9640 4250 50  0001 C CNN
-F 4 "AZ23C2V7" H 9640 4250 50  0001 C CNN "manf#"
-	1    9640 4250
-	1    0    0    -1
-$EndComp
-Wire Wire Line
-	7225 4515 7225 4455
+P 10570 4255
+F 0 "D4" H 10570 4471 50  0000 C CNN
+F 1 "AZ23C9V1" H 10570 4380 50  0000 C CNN
+F 2 "Package_TO_SOT_SMD:SOT-23" H 10570 4255 50  0001 C CNN
+F 3 "~" H 10570 4255 50  0001 C CNN
+F 4 "AZ23C2V7" H 10570 4255 50  0001 C CNN "manf#"
+	1    10570 4255
+	1    0    0    -1
+$EndComp
+Wire Wire Line
+	6705 4560 6705 4500
 Wire Wire Line
 	8095 4525 8095 4455
 Wire Wire Line
-	8895 4455 8895 4505
-Wire Wire Line
-	9640 4515 9640 4450
+	9425 4465 9425 4515
+Wire Wire Line
+	10570 4520 10570 4455
 $Comp
 L Device:R R9
@@
 	1    0    0    -1
 $EndComp
-Wire Wire Line
-	6790 3710 9990 3710
 $Comp
 L Connector_Generic:Conn_01x02 J1
@@
 $EndComp
 Wire Wire Line
-	6790 3610 9295 3610
-Wire Wire Line
-	6790 3510 9230 3510
-Wire Wire Line
-	6790 3410 8555 3410
-Wire Wire Line
-	6790 3310 8425 3310
-Wire Wire Line
-	6790 3210 7735 3210
-Wire Wire Line
-	6790 3110 7585 3110
-Wire Wire Line
-	6790 3010 6885 3010
-Wire Wire Line
-	6925 4255 6885 4255
-Wire Wire Line
-	6885 4255 6885 3010
-Wire Wire Line
-	7525 4255 7585 4255
-Wire Wire Line
-	7585 4255 7585 3110
-Connection ~ 7585 3110
-Wire Wire Line
-	7585 3110 10195 3110
+	6405 4300 6365 4300
+Wire Wire Line
+	7005 4300 7065 4300
 Wire Wire Line
 	7795 4255 7735 4255
 Wire Wire Line
-	7735 4255 7735 3210
-Connection ~ 7735 3210
-Wire Wire Line
-	7735 3210 10195 3210
-Wire Wire Line
 	8395 4255 8425 4255
 Wire Wire Line
-	8425 4255 8425 3310
-Connection ~ 8425 3310
-Wire Wire Line
-	8425 3310 10195 3310
-Wire Wire Line
-	8595 4255 8555 4255
-Wire Wire Line
-	8555 3410 8555 4255
-Connection ~ 8555 3410
-Wire Wire Line
-	8555 3410 10195 3410
-Wire Wire Line
-	9195 4255 9230 4255
-Wire Wire Line
-	9230 4255 9230 3510
-Connection ~ 9230 3510
-Wire Wire Line
-	9230 3510 10195 3510
-Wire Wire Line
-	9340 4250 9295 4250
-Wire Wire Line
-	9295 4250 9295 3610
-Connection ~ 9295 3610
-Wire Wire Line
-	9295 3610 10195 3610
-Wire Wire Line
-	9940 4250 9990 4250
-Wire Wire Line
-	9990 4250 9990 3710
-Connection ~ 9990 3710
-Wire Wire Line
-	9990 3710 10195 3710
-Wire Wire Line
-	10195 3010 6885 3010
-Connection ~ 6885 3010
+	9125 4265 9085 4265
+Wire Wire Line
+	9725 4265 9760 4265
+Wire Wire Line
+	10270 4255 10225 4255
+Wire Wire Line
+	10870 4255 10920 4255
 $Comp
 L Switch:SW_Push SW1
@@
 	6975 4725 6965 4725
 $Comp
-L Catwan_Farmer-rescue:ATSAMD21E18A-MU-Electronic_Cats-Catwan_Farmer-rescue-Catwan_Farmer-rescue-Catwan_Farmer-rescue U3
+L Catwan_Farmer-rescue:ATSAMD21E18A-MU-Electronic_Cats-Catwan_Farmer-rescue-Catwan_Farmer-rescue-Catwan_Farmer-rescue-Catwan_Farmer-rescue U3
 U 1 1 5E7C2C42
 P 2500 2160
@@
 $EndComp
 $Comp
-L Catwan_Farmer-rescue:74HC4052-Electronic_Cats-Catwan_Farmer-rescue-Catwan_Farmer-rescue-Catwan_Farmer-rescue U5
+L Catwan_Farmer-rescue:74HC4052-Electronic_Cats-Catwan_Farmer-rescue-Catwan_Farmer-rescue-Catwan_Farmer-rescue-Catwan_Farmer-rescue U5
 U 1 1 5E7C5328
 P 6390 3310
@@
 Wire Wire Line
 	3550 1380 3970 1380
+Wire Wire Line
+	6790 3010 6930 3010
+Wire Wire Line
+	6790 3110 6930 3110
+Wire Wire Line
+	6790 3210 6930 3210
+Wire Wire Line
+	6790 3310 6930 3310
+Wire Wire Line
+	6790 3410 6925 3410
+Wire Wire Line
+	6790 3510 6925 3510
+Wire Wire Line
+	6790 3610 6930 3610
+Wire Wire Line
+	6790 3710 6930 3710
+Text Label 6930 3010 0    50   ~ 0
+SENS_X1
+Text Label 6925 3410 0    50   ~ 0
+SENS_Y1
+Text Label 6930 3110 0    50   ~ 0
+SENS_X2
+Text Label 6925 3510 0    50   ~ 0
+SENS_Y2
+Text Label 6930 3210 0    50   ~ 0
+SENS_X3
+Text Label 6930 3310 0    50   ~ 0
+SENS_X4
+Text Label 6930 3610 0    50   ~ 0
+SENS_Y3
+Text Label 6930 3710 0    50   ~ 0
+SENS_Y4
+Wire Wire Line
+	10195 3010 9795 3010
+Wire Wire Line
+	10195 3110 9800 3110
+Wire Wire Line
+	10195 3210 9805 3210
+Wire Wire Line
+	10195 3310 9810 3310
+Wire Wire Line
+	10195 3410 9810 3410
+Wire Wire Line
+	10195 3510 9810 3510
+Wire Wire Line
+	10195 3610 9805 3610
+Wire Wire Line
+	10195 3710 9810 3710
+Text Label 9795 3010 0    50   ~ 0
+SENS_X1
+Text Label 9805 3210 0    50   ~ 0
+SENS_X2
+Text Label 9810 3410 0    50   ~ 0
+SENS_X3
+Text Label 9805 3610 0    50   ~ 0
+SENS_X4
+Text Label 9800 3110 0    50   ~ 0
+SENS_Y1
+Text Label 9810 3310 0    50   ~ 0
+SENS_Y2
+Text Label 9810 3510 0    50   ~ 0
+SENS_Y3
+Text Label 9810 3710 0    50   ~ 0
+SENS_Y4
+Text Label 6365 4300 3    50   ~ 0
+SENS_Y1
+Text Label 7065 4300 3    50   ~ 0
+SENS_X1
+Text Label 7735 4255 3    50   ~ 0
+SENS_Y2
+Text Label 8425 4255 3    50   ~ 0
+SENS_X2
+Text Label 9085 4265 3    50   ~ 0
+SENS_Y3
+Text Label 9760 4265 3    50   ~ 0
+SENS_X3
+Text Label 10225 4255 3    50   ~ 0
+SENS_Y4
+Text Label 10920 4255 3    50   ~ 0
+SENS_X4
 $EndSCHEMATC
