File: Hardware/Catwan_Farmer.kicad_pcb (KiCad board)
At the start: 2 copper layers, 60 x 70 mm, 56 parts, among them J1 SENSOR 1, J10 VSP, J2 SENSOR 2, J3 SENSOR 3, J4 BATT, J5 USB_B, J6 Conn_01x04, J7 DHT22, J9 SENSOR 4, SW1 SW_Push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

Commit message: 7HC40 and Diodes
Routing:
- net +3V3: track 0.00 -> 57.6 mm
- net Net-(D5-Pad2): track 0.00 -> 43.4 mm, vias 0 -> 2
- net Net-(D5-Pad1): track 0.00 -> 41.7 mm, vias 0 -> 2
- net /D+: track 0.00 -> 38.9 mm, vias 0 -> 2
- net /D-: track 0.00 -> 37.3 mm
- net /EN: track 0.00 -> 32.7 mm, vias 0 -> 2
- net Net-(D8-Pad2): track 0.00 -> 31.1 mm, vias 0 -> 2
- net /S0: track 0.00 -> 30.4 mm, vias 0 -> 2
- net Net-(D6-Pad1): track 0.00 -> 28.1 mm, vias 0 -> 2
- net Net-(D8-Pad1): track 0.00 -> 26.3 mm
- net Net-(D6-Pad2): track 0.00 -> 23.5 mm
- net /S1: track 0.00 -> 20.4 mm, vias 0 -> 2
- net Net-(D4-Pad2): track 0.00 -> 20.2 mm
- net Net-(D4-Pad1): track 0.00 -> 16.6 mm
- net /SENS_X: track 0.00 -> 14.8 mm, vias 0 -> 2
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
Commit message: routeo samd
Parts:
- moved SW1 23.4 mm to (120.4, 69.8)
- moved C11 1.29 mm to (134.8, 74.9), turned to 270 degrees
Routing:
- net /SENS_Y: track 14.2 -> 45.9 mm, vias 2 -> 3
- net Net-(SW1-Pad2): track 0.00 -> 27.1 mm, vias 0 -> 2
- net /ADC_BAT: track 1.95 -> 27.0 mm, vias 0 -> 2
- net GND: track 9.58 -> 34.6 mm, vias 2 -> 10
- net /SENS_X: track 14.8 -> 37.3 mm, vias 2 -> 3
- net /SWDIO: track 0.00 -> 15.3 mm, vias 0 -> 1
- net /SWCLK: track 0.00 -> 11.2 mm
- net Net-(C11-Pad2): track 0.00 -> 10.8 mm, vias 0 -> 2
- net +3V3: track 57.6 -> 58.5 mm

Commit message: delete tracks
Routing:
- net /SENS_Y: track 45.9 -> 0.00 mm, vias 3 -> 0
- net +3V3: track 58.5 -> 18.3 mm
- net /SENS_X: track 37.3 -> 0.00 mm, vias 3 -> 0
- net /EN: track 32.5 -> 0.00 mm, vias 2 -> 0
- net /S0: track 30.2 -> 0.00 mm, vias 2 -> 0
- net Net-(SW1-Pad2): track 27.1 -> 0.00 mm, vias 2 -> 0
- net /ADC_BAT: track 27.0 -> 0.00 mm, vias 2 -> 0
- net GND: track 34.6 -> 9.58 mm, vias 10 -> 2
- net /S1: track 20.4 -> 0.00 mm, vias 2 -> 0
- net /D-: track 37.3 -> 20.4 mm
- net /SWDIO: track 15.3 -> 0.00 mm, vias 1 -> 0
- net /SWCLK: track 11.2 -> 0.00 mm
- net Net-(C11-Pad2): track 10.8 -> 0.00 mm, vias 2 -> 0
- net /D+: track 39.1 -> 29.3 mm
- net /Y1: track 7.97 -> 0.00 mm
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
Commit message: RFM95
Parts:
- moved C7 12.9 mm to (164.7, 84.2)
- moved C12 12.4 mm to (149.7, 90.2)
- moved C9 12.4 mm to (159.0, 90.2)
- moved Y1 12.4 mm to (154.4, 90.2)
- moved R9 11.9 mm to (165.8, 79.6)
- moved D9 11.9 mm to (163.8, 79.6)
- moved U2 11.5 mm to (157.5, 59.9)
- moved R4 10.4 mm to (143.8, 75.7)
- moved R7 10.4 mm to (143.8, 77.6)
- moved U3 9.72 mm to (153.7, 79.8)
- moved C11 9.09 mm to (138.4, 83.2), turned to 0 degrees
- moved C3 7.91 mm to (138.4, 87.0)
- moved C8 7.91 mm to (138.4, 85.1)
- moved C5 6.22 mm to (138.3, 63.0)
- moved C1 6.22 mm to (141.2, 62.1)
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Routing:
- net +3V3: track 18.3 -> 90.4 mm, vias 0 -> 2
- net /EN: track 0.00 -> 52.7 mm, vias 0 -> 2
- net /DIO1: track 0.00 -> 42.3 mm, vias 0 -> 2
- net /DIO2: track 0.00 -> 40.4 mm, vias 0 -> 2
- net /DIO0: track 0.00 -> 39.1 mm, vias 0 -> 2
- net Net-(SW1-Pad2): track 0.00 -> 36.9 mm, vias 0 -> 2
- net /S1: track 0.00 -> 23.9 mm, vias 0 -> 2
- net /D-: track 20.4 -> 43.3 mm
- net /SWDIO: track 0.00 -> 19.7 mm
- net Net-(AE1-Pad1): track 0.00 -> 17.8 mm
- net /SWCLK: track 0.00 -> 16.8 mm
- net Net-(C11-Pad2): track 0.00 -> 16.3 mm, vias 0 -> 2
- net /D+: track 29.3 -> 43.3 mm, vias 2 -> 0
- net /DIO5: track 0.00 -> 12.8 mm
- net /Y1: track 0.00 -> 11.6 mm
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
Commit message: New routeo pcb
Routing:
- net +3V3: track 90.4 -> 187.7 mm, vias 2 -> 5
- net /BAT: track 0.00 -> 90.4 mm, vias 0 -> 2
- net GND: track 9.58 -> 71.6 mm, vias 2 -> 18
- net /SENS_Y: track 0.00 -> 50.6 mm, vias 0 -> 3
- net /SENS_X: track 0.00 -> 47.3 mm, vias 0 -> 2
- net VCC: track 0.00 -> 43.2 mm, vias 0 -> 2
- net /DHT_DAT: track 0.00 -> 41.3 mm, vias 0 -> 2
- net /S0: track 0.00 -> 38.6 mm, vias 0 -> 2
- net /ADC_BAT: track 0.00 -> 29.4 mm, vias 0 -> 2
- net Net-(D2-Pad2): track 0.00 -> 19.1 mm
- net +5V: track 0.00 -> 15.7 mm, vias 0 -> 1
- net Net-(R5-Pad1): track 0.00 -> 4.90 mm
- net Net-(R3-Pad2): track 0.00 -> 2.65 mm
- net /S1: track 23.9 -> 26.0 mm
- net Net-(D10-Pad1): track 0.00 -> 1.95 mm
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